File: hardware/I2CFEC.kicad_pcb (KiCad board)
At the start: 2 copper layers, 24 x 27.9 mm, 24 parts, among them J1 105444-0001, J2 B4B-XH-A, U1 PIC16F1454, U2 MIC2091

Commit message: Updated footprints
Parts:
- removed JP1: Jumper, Medo64:JP Dual (1205)
- added JP2: Jumper, Medo64:JP (0805), F.Cu at (24.7, 29.9)
- added JP2: Jumper, Medo64:JP (0805), F.Cu at (28.4, 29.9)
- U1: footprint Medo64:U Micro PIC16F1454 (SOIC-14) -> Medo64:U Micro [PIC16F1454] (SOIC-14)
- U2: footprint Medo64:U LoadSwitch MIC2091 (SOT23-5) -> Medo64:U LoadSwitch 100mA [MIC2091-1] (SOT23-5)
- VR1: footprint Medo64:VR Linear MCP1700 (SOT23-3) -> Medo64:VR Linear 3.3V 250mA [MCP1700] (SOT-23)
Connections:
- JP2 pad 1: 3V3 -> 3V3_USB
- JP2 pad 2: 3V3_USB -> 3V3
Routing:
- net 3V3_USB: track 25.5 -> 19.8 mm
- net VDD: track 36.8 -> 41.6 mm, vias 4 -> 3
- net 5V: track 16.0 -> 19.3 mm
- net POWER_FAULT: track 13.0 -> 13.8 mm
- net ICSP_VPP: track 11.0 -> 10.5 mm
Other:
- board text added: "GND"
- board text added: "SCL"
- board text added: "SDA"
- board text added: "V+"
